Commit message: update

File: src/manipulator/urdf/model.urdf.xacro (robot description, xacro)
@@ -195,7 +195,42 @@
         <material>Gazebo/Blue</material>
     </gazebo>
-    <ros2_control name="GazeboSystem" type="system">
+    <ros2_control name="RobotSystem" type="system">
         <hardware>
-            <!-- <plugin>gazebo_ros2_control/GazeboSystem</plugin> -->
+            <!-- Industrial Standard: Topic-Based Interface for External Bridges -->
+            <!-- This separates the ROS controller from your Python bridge -->
+            <plugin>topic_based_ros2_control/TopicBasedSystem</plugin>
+            <param name="joint_commands_topic">/hardware/motor_commands</param>
+            <param name="joint_states_topic">/hardware/motor_states</param>
+        </hardware>
+        <joint name="joint_1">
+            <command_interface name="position"/>
+            <state_interface name="position"/>
+            <state_interface name="velocity"/>
+        </joint>
+        <!-- Repeat for joints 2-5 -->
+        <joint name="joint_2">
+            <command_interface name="position"/>
+            <state_interface name="position"/>
+            <state_interface name="velocity"/>
+        </joint>
+        <joint name="joint_3">
+            <command_interface name="position"/>
+            <state_interface name="position"/>
+            <state_interface name="velocity"/>
+        </joint>
+        <joint name="joint_4">
+            <command_interface name="position"/>
+            <state_interface name="position"/>
+            <state_interface name="velocity"/>
+        </joint>
+        <joint name="joint_5">
+            <command_interface name="position"/>
+            <state_interface name="position"/>
+            <state_interface name="velocity"/>
+        </joint>
+    </ros2_control>
+    <!-- <ros2_control name="GazeboSystem" type="system">
+        <hardware>
+            <plugin>gazebo_ros2_control/GazeboSystem</plugin>
             <plugin>fake_components/GenericSystem</plugin>
         </hardware>
@@ -225,4 +260,4 @@
             <state_interface name="velocity"/>
         </joint>
-    </ros2_control>
+    </ros2_control> -->
 </robot>

Commit message: midchange

File: src/manipulator/urdf/model.urdf.xacro (robot description, xacro)
@@ -55,10 +55,17 @@
         <material>Gazebo/Black</material>
     </gazebo>
-    <joint name="joint_1" type="revolute">
+    <!-- <joint name="joint_1" type="revolute">
         <parent link="base_link"/>
         <child link="link_1"/>
         <origin rpy="0 0 0" xyz="0 0 0.1" />
         <axis xyz="0 0 1"/>
-        <limit effort="300" velocity="2.0" lower="-3.141593" upper="3.141593"/>
+        <limit effort="100" velocity="0.5" lower="-1.57" upper="1.57"/>
+    </joint> -->
+    <joint name="joint_1" type="continuous">
+        <parent link="base_link"/>
+        <child link="link_1"/>
+        <origin rpy="0 0 0" xyz="0 0 0.1" />
+        <axis xyz="0 0 1"/>
+        <limit effort="100" velocity="1.57"/>
     </joint>
     <link name="link_1">
@@ -88,5 +95,5 @@
         <origin rpy="0 -1.570796 0" xyz="-0.05 0 0.165" />
         <axis xyz="0 0 1"/>
-        <limit effort="300" velocity="2.0" lower="-3.141593" upper="3.141593"/>
+        <limit effort="100" velocity="0.5" lower="-1.57" upper="1.57"/>
     </joint>
     <link name="link_2">
@@ -116,5 +123,5 @@
         <origin rpy="0 0 0" xyz="0.41 0 0"/>
         <axis xyz="0 0 1"/>
-        <limit effort="300" velocity="2.0" lower="-3.141593" upper="3.141593"/>
+        <limit effort="100" velocity="0.5" lower="-1.57" upper="1.57"/>
     </joint>
     <link name="link_3">
@@ -144,5 +151,5 @@
         <origin rpy="0 0 0" xyz="0.43 0 0"/>
         <axis xyz="0 0 1"/>
-        <limit effort="300" velocity="2.0" lower="-3.141593" upper="3.141593"/>
+        <limit effort="100" velocity="0.5" lower="-1.57" upper="1.57"/>
     </joint>
     <link name="link_4">
@@ -172,5 +179,5 @@
         <origin rpy="0 1.570796 0" xyz="0.065 0 0.05"/>
         <axis xyz="0 0 1"/>
-        <limit effort="300" velocity="2.0" lower="-3.141593" upper="3.141593"/>
+        <limit effort="100" velocity="0.5" lower="-1.57" upper="1.57"/>
     </joint>
     <link name="link_5">

Commit message: update

File: src/manipulator/urdf/model.urdf.xacro (robot description, xacro)
@@ -67,5 +67,5 @@
         <origin rpy="0 0 0" xyz="0 0 0.1" />
         <axis xyz="0 0 1"/>
-        <limit effort="100" velocity="1.57"/>
+        <limit effort="100" velocity="1"/>
     </joint>
     <link name="link_1">
@@ -95,5 +95,5 @@
         <origin rpy="0 -1.570796 0" xyz="-0.05 0 0.165" />
         <axis xyz="0 0 1"/>
-        <limit effort="100" velocity="0.5" lower="-1.57" upper="1.57"/>
+        <limit effort="100" velocity="1" lower="-1.57" upper="1.57"/>
     </joint>
     <link name="link_2">
@@ -123,5 +123,5 @@
         <origin rpy="0 0 0" xyz="0.41 0 0"/>
         <axis xyz="0 0 1"/>
-        <limit effort="100" velocity="0.5" lower="-1.57" upper="1.57"/>
+        <limit effort="100" velocity="1" lower="-1.57" upper="1.57"/>
     </joint>
     <link name="link_3">
@@ -151,5 +151,5 @@
         <origin rpy="0 0 0" xyz="0.43 0 0"/>
         <axis xyz="0 0 1"/>
-        <limit effort="100" velocity="0.5" lower="-1.57" upper="1.57"/>
+        <limit effort="100" velocity="1" lower="-1.57" upper="1.57"/>
     </joint>
     <link name="link_4">
@@ -179,5 +179,5 @@
         <origin rpy="0 1.570796 0" xyz="0.065 0 0.05"/>
         <axis xyz="0 0 1"/>
-        <limit effort="100" velocity="0.5" lower="-1.57" upper="1.57"/>
+        <limit effort="100" velocity="1" lower="-1.57" upper="1.57"/>
     </joint>
     <link name="link_5">

Commit message: Updating

File: src/manipulator/urdf/model.urdf.xacro (robot description, xacro)
@@ -67,5 +67,5 @@
         <origin rpy="0 0 0" xyz="0 0 0.1" />
         <axis xyz="0 0 1"/>
-        <limit effort="100" velocity="1"/>
+        <limit effort="100" velocity="0.8727"/>
     </joint>
     <link name="link_1">
@@ -95,5 +95,5 @@
         <origin rpy="0 -1.570796 0" xyz="-0.05 0 0.165" />
         <axis xyz="0 0 1"/>
-        <limit effort="100" velocity="1" lower="-1.57" upper="1.57"/>
+        <limit effort="100" velocity="0.8727" lower="-1.57" upper="1.57"/>
     </joint>
     <link name="link_2">
@@ -123,5 +123,5 @@
         <origin rpy="0 0 0" xyz="0.41 0 0"/>
         <axis xyz="0 0 1"/>
-        <limit effort="100" velocity="1" lower="-1.57" upper="1.57"/>
+        <limit effort="100" velocity="0.8727" lower="-1.57" upper="1.57"/>
     </joint>
     <link name="link_3">
@@ -151,5 +151,5 @@
         <origin rpy="0 0 0" xyz="0.43 0 0"/>
         <axis xyz="0 0 1"/>
-        <limit effort="100" velocity="1" lower="-1.57" upper="1.57"/>
+        <limit effort="100" velocity="0.8727" lower="-1.57" upper="1.57"/>
     </joint>
     <link name="link_4">
@@ -179,5 +179,5 @@
         <origin rpy="0 1.570796 0" xyz="0.065 0 0.05"/>
         <axis xyz="0 0 1"/>
-        <limit effort="100" velocity="1" lower="-1.57" upper="1.57"/>
+        <limit effort="100" velocity="0.8727" lower="-1.57" upper="1.57"/>
     </joint>
     <link name="link_5">
